File: Hardware/BluetoothMate.sch (EAGLE design)
At the start: 27 parts, among them Q1 MOSFET-NCHANNELSMD, Q2 MOSFET-NCHANNELSMD, U1 BLUETOOTH-RN41, U3 V_REG_LDOSMD

Commit message: Updated Caps/Res to 0603 packages
Parts:
- C4: device SparkFun:CAP0402-CAP -> SparkFun:CAP0603-CAP
- R1, R2, R3, R4, R5, R6, R7, R8, R9: device SparkFun:RESISTOR0402-RES -> SparkFun:RESISTOR0603-RES

Commit message: Additional updates to layout
Parts:
- removed JP4: FIDUCIAL1X2.5, abes:FIDUCIAL1X2.5

Commit message: Fix silk screen/symbol errors
Parts:
- added U$2: REVISION, SparkFun-Aesthetics:REVISION
Other:
- note added: "J. Lindblom"
- note added: "T. Klopfenstein"
- note removed: "J. Lindblom, T. Klopfenstein"
Changed lines of the file:
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@@
 <part name="JP1" library="abes" deviceset="FIDUCIAL" device="1X2.5"/>
 <part name="LOGO1" library="SparkFun-Aesthetics" deviceset="OSHW-LOGO" device="S" value="OSHW-LOGOS"/>
+<part name="U$2" library="SparkFun-Aesthetics" deviceset="REVISION" device=""/>
 </parts>
 <sheets>
 <sheet>
 <plain>
-<text x="154.94" y="7.62" size="2.54" layer="97">J. Lindblom, T. Klopfenstein</text>
+<text x="171.704" y="11.43" size="2.54" layer="97">J. Lindblom</text>
 <text x="238.76" y="7.62" size="2.54" layer="97">v16</text>
+<text x="176.276" y="6.858" size="2.54" layer="97">T. Klopfenstein</text>
 </plain>
 <instances>
@@
 <instance part="JP1" gate="G$1" x="243.84" y="30.48"/>
 <instance part="LOGO1" gate="G$1" x="134.62" y="10.16"/>
+<instance part="U$2" gate="G$1" x="148.844" y="7.366"/>
 </instances>
 <busses>

Commit message: Added 2nd fiducial
Production files updated to v16a
Hardware files updated also
Parts:
- added JP4: FIDUCIAL1X2.5, abes:FIDUCIAL1X2.5
Changed lines of the file:
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@@
 <?xml version="1.0" encoding="utf-8"?>
 <!DOCTYPE eagle SYSTEM "eagle.dtd">
-<eagle version="6.4">
+<eagle version="6.5.0">
 <drawing>
 <settings>
@@
 <part name="LOGO1" library="SparkFun-Aesthetics" deviceset="OSHW-LOGO" device="S" value="OSHW-LOGOS"/>
 <part name="U$2" library="SparkFun-Aesthetics" deviceset="REVISION" device=""/>
+<part name="JP4" library="abes" deviceset="FIDUCIAL" device="1X2.5"/>
 </parts>
 <sheets>
@@
 <instance part="JP3" gate="G$1" x="33.02" y="88.9"/>
 <instance part="TP1" gate="G$1" x="91.44" y="167.64"/>
-<instance part="JP1" gate="G$1" x="243.84" y="30.48"/>
+<instance part="JP1" gate="G$1" x="243.84" y="27.94"/>
 <instance part="LOGO1" gate="G$1" x="134.62" y="10.16"/>
 <instance part="U$2" gate="G$1" x="148.844" y="7.366"/>
+<instance part="JP4" gate="G$1" x="243.84" y="33.02"/>
 </instances>
 <busses>
